Commit message: Assignment 1 on gazebo

File: catkin_ws/src/demo_bot_gazebo/urdf/my_robot.urdf (robot description, URDF)
Before this commit: robot test_robot, 1 links, 0 joints
Links:
- added link base_footprint, mass 0.0001; visual box size=0.001 0.001 0.001
- added link caster_back_link, mass 0.5; collision sphere radius=0.025; visual sphere radius=0.025
- added link caster_front_link, mass 0.5; collision sphere radius=0.025; visual sphere radius=0.025
- added link front_left_wheel, mass 2.5; collision cylinder length=0.02 radius=0.04; visual cylinder length=0.02 radius=0.04
- added link front_right_wheel, mass 2.5; collision cylinder length=0.02 radius=0.04; visual cylinder length=0.02 radius=0.04
- added link hokuyo_link; visual box size=0.05 0.05 0.05
- link base_link: geometry collision cylinder length=0.02 radius=0.15; visual cylinder length=0.02 radius=0.15
Joints:
- added joint base_footprint_joint: type fixed, parent base_footprint, child base_link, origin xyz=0 0 0.04 rpy=0 0 0
- added joint caster_back_joint: type fixed, parent base_link, child caster_back_link, origin xyz=-0.135 0.0 0.009 rpy=-1.57079632679 0 0
- added joint caster_front_joint: type fixed, parent base_link, child caster_front_link, origin xyz=0.115 0.0 0.007 rpy=-1.57079632679 0 0
- added joint front_left_wheel_joint: type continuous, parent base_link, child front_left_wheel, origin xyz=0.0 -0.15 0.0 rpy=0 0 0, axis 0 1 0, limit effort=100 velocity=100
- added joint front_right_wheel_joint: type continuous, parent base_link, child front_right_wheel, origin xyz=0.0 0.15 0.0 rpy=0 0 0, axis 0 1 0, limit effort=100 velocity=100
- added joint hokuyo_joint: type fixed, parent base_link, child hokuyo_link, origin xyz=0.125 0 0.0325 rpy=0 0 0
